File: Hardware/RP488.kicad_sch (KiCad schematic)
At the start: 33 parts, among them J1 GPIB, J2 SWD, J3 USB Mini, U1 SN75160, U2 SN75161, U3 RP2354A, U5 USBLC6-2SC6, U6 LD3985M33R_SOT23

Commit message: Renamed directory, added PNG of schematic and PCB 3d view
Parts:
- D1: value LED -> Activity
- D2: value LED -> Error
- L1: value L -> 3u3
Changed lines of the file:
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@@
 		(in_pos_files yes)
 		(dnp no)
-		(fields_autoplaced yes)
 		(property "Reference" "R3"
-			(at 64.77 67.31 90)
+			(at 64.516 71.374 90)
 			(show_name no)
 			(do_not_autoplace no)
@@
 		)
 		(property "Value" "27R"
-			(at 64.77 69.85 90)
+			(at 65.024 76.2 90)
 			(show_name no)
 			(do_not_autoplace no)
@@
 		(in_pos_files yes)
 		(dnp no)
-		(fields_autoplaced yes)
 		(property "Reference" "R5"
-			(at 177.8 139.7 90)
+			(at 177.8 143.51 90)
 			(show_name no)
 			(do_not_autoplace no)
@@
 		)
 		(property "Value" "1K"
-			(at 177.8 142.24 90)
+			(at 177.8 148.59 90)
 			(show_name no)
 			(do_not_autoplace no)
@@
 		(in_pos_files yes)
 		(dnp no)
-		(fields_autoplaced yes)
 		(property "Reference" "L1"
-			(at 124.46 41.9099 0)
+			(at 123.444 34.544 0)
 			(show_name no)
 			(do_not_autoplace no)
@@
 			)
 		)
-		(property "Value" "L"
-			(at 124.46 44.4499 0)
+		(property "Value" "3u3"
+			(at 123.19 36.576 0)
 			(show_name no)
 			(do_not_autoplace no)
@@
 		(in_pos_files yes)
 		(dnp no)
-		(fields_autoplaced yes)
 		(property "Reference" "R2"
-			(at 64.77 95.25 90)
+			(at 64.77 99.314 90)
 			(show_name no)
 			(do_not_autoplace no)
@@
 		)
 		(property "Value" "27R"
-			(at 64.77 97.79 90)
+			(at 64.77 104.14 90)
 			(show_name no)
 			(do_not_autoplace no)
@@
 		(in_pos_files yes)
 		(dnp no)
-		(fields_autoplaced yes)
 		(property "Reference" "R6"
-			(at 177.8 147.32 90)
+			(at 177.546 151.384 90)
 			(show_name no)
 			(do_not_autoplace no)
@@
 		)
 		(property "Value" "1K"
-			(at 177.8 149.86 90)
+			(at 177.8 156.21 90)
 			(show_name no)
 			(do_not_autoplace no)
@@
 		(dnp no)
 		(property "Reference" "D1"
-			(at 170.4975 139.7 0)
+			(at 168.91 140.97 0)
 			(show_name no)
 			(do_not_autoplace no)
@@
 			)
 		)
-		(property "Value" "LED"
-			(at 170.4975 142.24 0)
+		(property "Value" "Activity"
+			(at 168.91 143.256 0)
 			(show_name no)
 			(do_not_autoplace no)
@@
 		(dnp no)
 		(property "Reference" "D2"
-			(at 170.4975 147.32 0)
+			(at 168.91 156.718 0)
 			(show_name no)
 			(do_not_autoplace no)
@@
 			)
 		)
-		(property "Value" "LED"
-			(at 170.4975 149.86 0)
+		(property "Value" "Error"
+			(at 169.164 159.004 0)
 			(show_name no)
 			(do_not_autoplace no)
